Commit message: Update: addes the Isaac Sim package and the module_2 folder with updated SHL-1 USD

File: ros2_ws/src/rse_shl1_description/urdf/shl1_robot.urdf.xacro (robot description, xacro)
@@ -79,5 +79,5 @@
       <xacro:unless value="${y > 0}"><origin xyz="0 -0.1 0" rpy="0 0 0"/></xacro:unless>
       <axis xyz="0 0 1"/>
-      <limit lower="-0.785398" upper="0.785398" effort="20" velocity="6.28"/>
+      <limit lower="-1.5708" upper="1.5708" effort="20" velocity="6.28"/>
       <dynamics damping="${STEER_D}"/>
     </joint>
